File: KiCAD/S11639-01_SPIboard.kicad_sch (KiCad schematic)
At the start: 60 parts, among them IC1 74LVC1T45GW,125, IC2 74LVC1T45GW,125, IC3 74LVC1T45GW,125, IC4 MCP33131D-10-I_MS, IC5 74LVC1T45GW,125, J1 Conn_01x03_Male, J2 Conn_02x10_Odd_Even, J3 705430001, J4 Conn_01x03_Male, U1 ADA4807-2ARMZ-R7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

Commit message: Add files via upload
Parts:
- C14, C9: Digikey 399-C0603C102F3GAC7867CT-ND -> 311-1743-1-ND
Changed lines of the file:
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@@
       (effects (font (size 1.27 1.27)) hide)
     )
-    (property "Digikey" "399-C0603C102F3GAC7867CT-ND" (id 4) (at 161.544 210.312 0)
-      (effects (font (size 1.27 1.27)) hide)
-    )
-    (property "Description" "CAP CER 1000PF 25V C0G/NP0 0603" (id 5) (at 161.544 210.312 0)
+    (property "Digikey" "311-1743-1-ND" (id 4) (at 161.544 210.312 0)
+      (effects (font (size 1.27 1.27)) hide)
+    )
+    (property "Description" "CAP CER 1000PF 50V C0G/NPO 0603" (id 5) (at 161.544 210.312 0)
       (effects (font (size 1.27 1.27)) hide)
     )
@@
       (effects (font (size 1.27 1.27)) hide)
     )
-    (property "Digikey" "399-C0603C102F3GAC7867CT-ND" (id 4) (at 128.524 210.312 0)
-      (effects (font (size 1.27 1.27)) hide)
-    )
-    (property "Description" "CAP CER 1000PF 25V C0G/NP0 0603" (id 5) (at 128.524 210.312 0)
-      (effects (font (size 1.27 1.27)) hide)
-    )
+    (property "Digikey" "311-1743-1-ND" (id 4) (at 128.524 210.312 0)
+      (effects (font (size 1.27 1.27)) hide)
+    )
+    (property "Description" "CAP CER 1000PF 50V C0G/NPO 0603" (id 5) (at 128.524 210.312 0)
+      (effects (font (size 1.27 1.27)) hide)
+    )
