File: KiCAD/S11639-01_SPIboard.kicad_pcb (KiCad board)
At the start: 4 copper layers, 70 x 40 mm, 60 parts, among them IC1 74LVC1T45GW,125, IC2 74LVC1T45GW,125, IC3 74LVC1T45GW,125, IC4 MCP33131D-10-I_MS, IC5 74LVC1T45GW,125, J1 Conn_01x03_Male, J2 Conn_02x10_Odd_Even, J3 705430001, J4 Conn_01x03_Male, U1 ADA4807-2ARMZ-R7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

Commit message: Add files via upload
Changed lines of the file:
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@@
     (descr "Capacitor SMD 0603 (1608 Metric), square (rectangular) end terminal, IPC_7351 nominal, (Body size source: IPC-SM-782 page 76, https://www.pcb-3d.com/wordpress/wp-content/uploads/ipc-sm-782a_amendment_1_and_2.pdf), generated with kicad-footprint-generator")
     (tags "capacitor")
-    (property "Description" "CAP CER 1000PF 25V C0G/NP0 0603")
-    (property "Digikey" "399-C0603C102F3GAC7867CT-ND")
+    (property "Description" "CAP CER 1000PF 50V C0G/NPO 0603")
+    (property "Digikey" "311-1743-1-ND")
     (property "Sheetfile" "S11639-01_SPIboard.kicad_sch")
     (property "Sheetname" "")
@@
     (descr "Capacitor SMD 0603 (1608 Metric), square (rectangular) end terminal, IPC_7351 nominal, (Body size source: IPC-SM-782 page 76, https://www.pcb-3d.com/wordpress/wp-content/uploads/ipc-sm-782a_amendment_1_and_2.pdf), generated with kicad-footprint-generator")
     (tags "capacitor")
-    (property "Description" "CAP CER 1000PF 25V C0G/NP0 0603")
-    (property "Digikey" "399-C0603C102F3GAC7867CT-ND")
+    (property "Description" "CAP CER 1000PF 50V C0G/NPO 0603")
+    (property "Digikey" "311-1743-1-ND")
     (property "Sheetfile" "S11639-01_SPIboard.kicad_sch")
     (property "Sheetname" "")
@@
     (property "Sheetname" "")
     (attr through_hole)
-    (fp_text reference "J3" (at 4.81 2.6) (layer "F.SilkS")
+    (fp_text reference "J3" (at -0.855 -5.125) (layer "F.SilkS")
       (effects (font (size 1 1) (thickness 0.15)))
     )
@@
       (effects (font (size 1 1) (thickness 0.15)))
     )
+    (fp_line (start 3.685 2.54) (end -3.685 2.54) (layer "F.SilkS") (width 0.127))
     (fp_line (start -3.685 2.54) (end -3.685 -4.06) (layer "F.SilkS") (width 0.127))
     (fp_line (start -3.685 -4.06) (end 3.685 -4.06) (layer "F.SilkS") (width 0.127))
-    (fp_line (start 3.685 2.54) (end -3.685 2.54) (layer "F.SilkS") (width 0.127))
     (fp_line (start 3.685 -4.06) (end 3.685 2.54) (layer "F.SilkS") (width 0.127))
     (fp_circle (center 4.28 0) (end 4.38 0) (layer "F.SilkS") (width 0.2) (fill none))
     (fp_line (start 3.935 -4.31) (end 3.935 2.79) (layer "F.CrtYd") (width 0.05))
+    (fp_line (start -3.935 -4.31) (end 3.935 -4.31) (layer "F.CrtYd") (width 0.05))
+    (fp_line (start -3.935 2.79) (end -3.935 -4.31) (layer "F.CrtYd") (width 0.05))
     (fp_line (start 3.935 2.79) (end -3.935 2.79) (layer "F.CrtYd") (width 0.05))
-    (fp_line (start -3.935 2.79) (end -3.935 -4.31) (layer "F.CrtYd") (width 0.05))
-    (fp_line (start -3.935 -4.31) (end 3.935 -4.31) (layer "F.CrtYd") (width 0.05))
     (fp_line (start 3.685 -4.06) (end 3.685 2.54) (layer "F.Fab") (width 0.127))
     (fp_line (start 3.685 2.54) (end -3.685 2.54) (layer "F.Fab") (width 0.127))

Commit message: Version 0.2, tested
Tested, noise is 0.5mV in , per spec for the part.  See the firmware directory for an Arduino sketch to use the board.   See the Teensy Carrier for a mating board that hosts a Teensy 4.0 to run the sensor.
Connections:
- R5 pad 1: Net-(C16-Pad2) -> Net-(C16-Pad1)
Routing:
- net Net-(C16-Pad1): track 3.78 -> 8.58 mm
- net Net-(C16-Pad2): track 11.9 -> 7.93 mm
Other:
- board text added: "S11639-01 Sensor, 16bit ADC, SPI Rev 0.2 Mitchell C Nelson, PhD (c) 2023, 2024"
- board text removed: "S11639-01 Sensor, 16bit ADC, SPI Mitchell C Nelson, PhD (c) 2023"
Changed lines of the file:
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@@
     (property "Sheetname" "")
     (attr through_hole)
-    (fp_text reference "J3" (at -0.855 -5.125) (layer "F.SilkS")
-      (effects (font (size 1 1) (thickness 0.15)))
+    (fp_text reference "J3" (at 4.46 -3.72) (layer "F.SilkS")
+      (effects (font (size 0.66 0.66) (thickness 0.1)))
     )
     (fp_text value "705430001" (at 5.605 3.558) (layer "F.Fab")
@@
     (fp_line (start 0.8 0.4125) (end -0.8 0.4125) (layer "F.Fab") (width 0.1))
     (pad "1" smd roundrect (at -0.825 0 90) (size 0.8 0.95) (layers "F.Cu" "F.Paste" "F.Mask") (roundrect_rratio 0.25)
-      (net 10 "Net-(C16-Pad2)") (pintype "passive"))
+      (net 9 "Net-(C16-Pad1)") (pintype "passive"))
     (pad "2" smd roundrect (at 0.825 0 90) (size 0.8 0.95) (layers "F.Cu" "F.Paste" "F.Mask") (roundrect_rratio 0.25)
       (net 8 "Net-(C14-Pad1)") (pintype "passive"))
@@
     (effects (font (size 0.6 0.6) (thickness 0.1)))
   )
-  (gr_text "S11639-01 Sensor, 16bit ADC, SPI\nMitchell C Nelson, PhD (c) 2023" (at 111.45 117.53) (layer "F.SilkS")
+  (gr_text "S11639-01 Sensor, 16bit ADC, SPI Rev 0.2\nMitchell C Nelson, PhD (c) 2023, 2024" (at 112.5 117.53) (layer "F.SilkS")
     (effects (font (size 0.8 0.8) (thickness 0.14)))
   )
@@
   (segment (start 149.13 103.2) (end 153.47 103.2) (width 0.25) (layer "B.Cu") (net 5))
   (segment (start 132.04 110.12) (end 128.3 110.12) (width 0.25) (layer "B.Cu") (net 5))
+  (segment (start 156.425 107.79) (end 156.905 107.31) (width 0.25) (layer "F.Cu") (net 6))
   (segment (start 157.58 104.25) (end 156.885 104.945) (width 0.25) (layer "F.Cu") (net 6))
   (segment (start 153.615 97.1) (end 153.595 97.12) (width 0.25) (layer "F.Cu") (net 6))
   (segment (start 153.57 95.355) (end 153.615 95.4) (width 0.25) (layer "F.Cu") (net 6))
   (segment (start 156.885 105.64) (end 156.885 107.29) (width 0.25) (layer "F.Cu") (net 6))
+  (segment (start 155.3225 107.79) (end 156.425 107.79) (width 0.25) (layer "F.Cu") (net 6))
   (segment (start 155.15 97.12) (end 155.29 96.98) (width 0.25) (layer "F.Cu") (net 6))
   (segment (start 153.615 95.4) (end 153.615 97.1) (width 0.25) (layer "F.Cu") (net 6))
-  (segment (start 156.545 107.67) (end 156.905 107.31) (width 0.25) (layer "F.Cu") (net 6))
-  (segment (start 155.4425 107.67) (end 156.545 107.67) (width 0.25) (layer "F.Cu") (net 6))
+  (segment (start 154.93 108.1825) (end 155.3225 107.79) (width 0.25) (layer "F.Cu") (net 6))
   (segment (start 156.885 104.945) (end 156.885 105.64) (width 0.25) (layer "F.Cu") (net 6))
   (segment (start 153.595 97.12) (end 155.15 97.12) (width 0.25) (layer "F.Cu") (net 6))
   (segment (start 156.885 107.29) (end 156.905 107.31) (width 0.25) (layer "F.Cu") (net 6))
-  (segment (start 154.93 108.1825) (end 155.4425 107.67) (width 0.25) (layer "F.Cu") (net 6))
   (segment (start 153.57 93.86) (end 153.57 95.355) (width 0.25) (layer "F.Cu") (net 6))
   (via (at 157.58 104.25) (size 1) (drill 0.5) (layers "F.Cu" "B.Cu") (free) (net 6))
@@
   (segment (start 156.9275 108.8325) (end 157.01 108.915) (width 0.25) (layer "F.Cu") (net 9))
   (segment (start 157.01 108.915) (end 158.59 108.915) (width 0.25) (layer "F.Cu") (net 9))
+  (segment (start 153.49 108.5) (end 153.49 107.72) (width 0.25) (layer "F.Cu") (net 9))
+  (segment (start 154.26 107.34) (end 154.57 107.34) (width 0.25) (layer "F.Cu") (net 9))
+  (segment (start 154.57 107.34) (end 155.1575 106.7525) (width 0.25) (layer "F.Cu") (net 9))
+  (segment (start 155.1575 106.7525) (end 155.1575 106.3825) (width 0.25) (layer "F.Cu") (net 9))
+  (segment (start 153.49 107.72) (end 153.87 107.34) (width 0.25) (layer "F.Cu") (net 9))
   (segment (start 158.59 108.915) (end 158.65 108.975) (width 0.25) (layer "F.Cu") (net 9))
+  (segment (start 153.87 107.34) (end 154.26 107.34) (width 0.25) (layer "F.Cu") (net 9))
+  (segment (start 154.93 108.8325) (end 153.8225 108.8325) (width 0.25) (layer "F.Cu") (net 9))
+  (segment (start 153.8225 108.8325) (end 153.49 108.5) (width 0.25) (layer "F.Cu") (net 9))
   (segment (start 154.93 108.8325) (end 156.9275 108.8325) (width 0.25) (layer "F.Cu") (net 9))
   (segment (start 158.61 110.565) (end 158.65 110.525) (width 0.25) (layer "F.Cu") (net 10))
   (segment (start 153.355 109.6675) (end 153.54 109.4825) (width 0.25) (layer "F.Cu") (net 10))
-  (segment (start 153.26 109.2025) (end 153.54 109.4825) (width 0.25) (layer "F.Cu") (net 10))
-  (segment (start 155.1575 106.3825) (end 153.26 108.28) (width 0.25) (layer "F.Cu") (net 10))
   (segment (start 153.54 109.4825) (end 154.93 109.4825) (width 0.25) (layer "F.Cu") (net 10))
-  (segment (start 153.26 108.28) (end 153.26 109.2025) (width 0.25) (layer "F.Cu") (net 10))
   (segment (start 157.01 110.565) (end 158.61 110.565) (width 0.25) (layer "F.Cu") (net 10))
   (segment (start 154.93 109.4825) (end 155.9275 109.4825) (width 0.25) (layer "F.Cu") (net 10))
